File: MFA_I2C/MFA_I2C.kicad_pcb (KiCad board)
At the start: 2 copper layers, 22 parts, among them J1 DIN41612_02x32_AC, J2 Conn_02x04_Odd_Even, SW1 Terminate, SW2 ADR, SW3 INT, U1 74LS00, U2 74LS85, U3 PCF8584, X1 ACO-3MHz-A

Commit message: changed
Parts:
- added H1: MountingHole_Pad, MountingHole:MountingHole_3.2mm_M3_ISO14580_Pad, F.Cu at (78.0, 126.6)
- added H2: MountingHole_Pad, MountingHole:MountingHole_3.2mm_M3_ISO14580_Pad, F.Cu at (231.4, 126.5)
- added H3: MountingHole_Pad, MountingHole:MountingHole_3.2mm_M3_ISO14580_Pad, F.Cu at (78.0, 37.3)
- added H4: MountingHole_Pad, MountingHole:MountingHole_3.2mm_M3_ISO14580_Pad, F.Cu at (231.4, 37.6)
- added J3: Conn_01x05, Connector_PinHeader_2.54mm:PinHeader_1x05_P2.54mm_Vertical, F.Cu at (179.3, 55.4)
- C1: value 10nF -> 0.1uF; footprint Capacitor_THT:CP_Radial_D4.0mm_P2.00mm -> Capacitor_THT:C_Rect_L4.6mm_W2.0mm_P2.50mm_MKS02_FKP02
- C2: value 15pF -> 0.1uF
- C4: value 0.1uF -> 10nF; footprint Capacitor_THT:C_Rect_L4.6mm_W2.0mm_P2.50mm_MKS02_FKP02 -> Capacitor_THT:CP_Radial_D4.0mm_P2.00mm
- C5: value 0.1uF -> 15pF
- J2: value Conn_02x04_Odd_Even -> Conn_02x03_Odd_Even; footprint Connector_IDC:IDC-Header_2x04_P2.54mm_Horizontal -> Connector_IDC:IDC-Header_2x03_P2.54mm_Horizontal
- SW1: value Terminate -> ADR; footprint Button_Switch_THT:SW_DIP_SPSTx03_Slide_9.78x9.8mm_W7.62mm_P2.54mm -> Button_Switch_THT:SW_DIP_SPSTx04_Slide_9.78x12.34mm_W7.62mm_P2.54mm
- SW2: value ADR -> INT; footprint Button_Switch_THT:SW_DIP_SPSTx04_Slide_9.78x12.34mm_W7.62mm_P2.54mm -> Button_Switch_THT:SW_DIP_SPSTx06_Slide_9.78x17.42mm_W7.62mm_P2.54mm
- SW3: value INT -> Terminate; footprint Button_Switch_THT:SW_DIP_SPSTx06_Slide_9.78x17.42mm_W7.62mm_P2.54mm -> Button_Switch_THT:SW_DIP_SPSTx03_Slide_9.78x9.8mm_W7.62mm_P2.54mm
- moved J1 190.5 mm to (228.9, 42.7), turned to -90 degrees
- moved U2 142.4 mm to (210.4, 121.1), turned to 180 degrees
- moved U1 103.0 mm to (185.0, 67.4)
- moved C5 97.1 mm to (172.3, 42.1), turned to -90 degrees
- moved J2 91.3 mm to (85.3, 73.2), turned to 180 degrees
- moved SW2 85.2 mm to (186.3, 87.1), turned to 90 degrees
- moved C3 83.1 mm to (179.3, 47.8), turned to -90 degrees
- moved R6 79.9 mm to (93.0, 39.5)
- moved R7 79.9 mm to (96.8, 39.5)
- moved R1 70.2 mm to (167.3, 110.9), turned to -90 degrees
- moved R2 68.9 mm to (171.1, 110.9), turned to -90 degrees
- moved C2 68.8 mm to (202.1, 126.2), turned to 180 degrees
- moved R3 68.0 mm to (174.9, 110.9), turned to -90 degrees
- moved R4 67.5 mm to (178.7, 110.9), turned to -90 degrees
- moved U3 63.5 mm to (185.0, 52.8), turned to 90 degrees
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Connections:
- C2 pad 1: /CLK_{I2C} -> VCC
- C5 pad 1: VCC -> /CLK_{I2C}
- J2 pad 2: VCC -> /~{INT_{I2C}}
- J2 pad 4: /SCL -> GND
- J2 pad 5: /~{INT_{I2C}} -> /SCL
- J2 pad 6: unconnected-(J2-Pad6) -> GND
- R5 pad 2: Net-(R5-Pad2) -> /~{INT}
- R8 pad 2: /~{INT} -> Net-(R8-Pad2)
- SW1 pad 1: /SDA -> GND
- SW1 pad 2: /SCL -> GND
- SW1 pad 3: /~{INT_{I2C}} -> GND
- SW1 pad 4: Net-(R7-Pad2) -> GND
- SW1 pad 5: Net-(R6-Pad2) -> /B_{7}
- SW1 pad 6: Net-(R5-Pad2) -> /B_{6}
- SW2 pad 1: GND -> /RST_{5.5}
- SW2 pad 2: GND -> /RST_{6.5}
- SW2 pad 3: GND -> /RST_{7.5}
- SW2 pad 4: GND -> /RST_{5.5}
- SW2 pad 5: /B_{7} -> /RST_{6.5}
- SW2 pad 6: /B_{6} -> /RST_{7.5}
- SW2 pad 7: /B_{5} -> /INT
- SW2 pad 8: /B_{4} -> /INT
- SW3 pad 1: /RST_{5.5} -> /SDA
- SW3 pad 2: /RST_{6.5} -> /SCL
- SW3 pad 3: /RST_{7.5} -> /~{INT_{I2C}}
- SW3 pad 4: /RST_{5.5} -> Net-(R8-Pad2)
- SW3 pad 5: /RST_{6.5} -> Net-(R7-Pad2)
- SW3 pad 6: /RST_{7.5} -> Net-(R6-Pad2)
- U1 pad 11: Net-(SW3-Pad7) -> /IOWR
- U1 pad 12: /~{INT_{I2C}} -> /~{IOR}
- U1 pad 13: /~{INT_{I2C}} -> /~{IOW}
- U1 pad 4: /~{IOR} -> /~{INT_{I2C}}
- U1 pad 5: /~{IOW} -> /~{INT_{I2C}}
- U1 pad 6: /IOWR -> /INT_{I2C}
- U1 pad 8: Net-(SW3-Pad10) -> /INT
Routing:
- net VCC: track 0.00 -> 330.0 mm
- net /~{INT_{I2C}}: track 0.00 -> 98.3 mm
- net /SCL: track 0.00 -> 84.8 mm
- net /SDA: track 0.00 -> 80.5 mm
- net /IOWR: track 0.00 -> 79.2 mm, vias 0 -> 1
- net /~{IOW}: track 0.00 -> 75.1 mm, vias 0 -> 1
- net /~{IOR}: track 0.00 -> 72.9 mm, vias 0 -> 1
- net /a=b: track 0.00 -> 65.4 mm, vias 0 -> 1
- net /~{RESOUT}: track 0.00 -> 58.9 mm, vias 0 -> 1
- net /RST_{5.5}: track 0.00 -> 57.2 mm, vias 0 -> 1
- net /RST_{6.5}: track 0.00 -> 57.1 mm, vias 0 -> 1
- net /RST_{7.5}: track 0.00 -> 55.7 mm, vias 0 -> 1
- net /A_{0}: track 0.00 -> 55.0 mm, vias 0 -> 1
- net /A_{7}: track 0.00 -> 48.8 mm
- net /B_{4}: track 0.00 -> 48.5 mm
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- added copper zone on B.Cu, net GND
- added copper zone on F.Cu, net GND
Other:
- board outline added: 160 x 100.1 mm
- board text added: "+5V"
- board text added: "GND"
- board text added: "SDA"
- board text added: "~{INT_{I2C}}"

Commit message: next version
Parts:
- removed J2: Conn_02x03_Odd_Even, Connector_IDC:IDC-Header_2x03_P2.54mm_Horizontal
- removed the J3 at (179.3, 55.4)
- added BT1: CR2032, Battery:BatteryHolder_Keystone_103_1x20mm, F.Cu at (118.4, 96.5)
- added C12: 4.7uF, Capacitor_THT:C_Radial_D4.0mm_H5.0mm_P1.50mm, F.Cu at (186.3, 73.2)
- added C13: 4.7uF, Capacitor_THT:C_Radial_D4.0mm_H5.0mm_P1.50mm, F.Cu at (186.3, 90.9)
- added C4: 0.1uF, Capacitor_THT:C_Rect_L4.6mm_W2.0mm_P2.50mm_MKS02_FKP02, F.Cu at (209.8, 101.1)
- added C5: 0.1uF, Capacitor_THT:C_Rect_L4.6mm_W2.0mm_P2.50mm_MKS02_FKP02, F.Cu at (186.9, 60.5)
- added C6: 0.1uF, Capacitor_THT:C_Rect_L4.6mm_W2.0mm_P2.50mm_MKS02_FKP02, F.Cu at (186.9, 78.2)
- added C7: 0.1uF, Capacitor_THT:C_Rect_L4.6mm_W2.0mm_P2.50mm_MKS02_FKP02, F.Cu at (145.0, 80.8)
- added C8: 0.1uF, Capacitor_THT:C_Rect_L4.6mm_W2.0mm_P2.50mm_MKS02_FKP02, F.Cu at (145.0, 98.6)
- added J1: Conn_01x05, Connector_PinHeader_2.54mm:PinHeader_1x05_P2.54mm_Vertical, F.Cu at (144.4, 47.8)
- added J4: C-Control, Connector_IDC:IDC-Header_2x03_P2.54mm_Horizontal, F.Cu at (85.3, 58.5)
- added J5: JST-PH, Connector_JST:JST_PH_S5B-PH-K_1x05_P2.00mm_Horizontal, F.Cu at (78.3, 74.2)
- added J6: JST-PH, Connector_JST:JST_PH_S5B-PH-K_1x05_P2.00mm_Horizontal, F.Cu at (78.2, 87.6)
- added J7: Grove/Seed, Connector_JST:JST_PH_S4B-PH-K_1x04_P2.00mm_Horizontal, F.Cu at (78.2, 101.9)
- added J8: Grove/Seed, Connector_JST:JST_PH_S4B-PH-K_1x04_P2.00mm_Horizontal, F.Cu at (78.2, 113.3)
- added RN1: 5k6, Resistor_THT:R_Array_SIP9, F.Cu at (159.0, 109.3)
- added SW4: Master INT, Button_Switch_THT:SW_DIP_SPSTx05_Slide_9.78x14.88mm_W7.62mm_P2.54mm, F.Cu at (161.5, 103.6)
- added SW5: address, Button_Switch_THT:SW_DIP_SPSTx03_Slide_9.78x9.8mm_W7.62mm_P2.54mm, F.Cu at (127.2, 78.3)
- added U4: 74LS04, Package_DIP:DIP-14_W7.62mm_Socket, F.Cu at (190.7, 103.6)
- added U5: 74LS00, Package_DIP:DIP-14_W7.62mm_Socket, F.Cu at (190.8, 68.1)
- added U6: 74LS00, Package_DIP:DIP-14_W7.62mm_Socket, F.Cu at (190.7, 85.8)
- added U7: 24LC64, Package_DIP:DIP-8_W7.62mm_Socket, F.Cu at (133.6, 85.9)
- added U8: DS1307+, Package_DIP:DIP-8_W7.62mm_Socket, F.Cu at (133.6, 103.6)
- added Y1: 32.768 kHz, Crystal:Crystal_C38-LF_D3.0mm_L8.0mm_Horizontal_1EP_style2, F.Cu at (133.9, 107.9)
- R1, R2, R3, R4: value 4k7 -> 10k; footprint Resistor_THT:R_Axial_DIN0207_L6.3mm_D2.5mm_P10.16mm_Horizontal -> Resistor_THT:R_Axial_DIN0207_L6.3mm_D2.5mm_P7.62mm_Horizontal
- R5, R6, R7, R8: footprint Resistor_THT:R_Axial_DIN0207_L6.3mm_D2.5mm_P10.16mm_Horizontal -> Resistor_THT:R_Axial_DIN0207_L6.3mm_D2.5mm_P7.62mm_Horizontal
- SW1: value ADR -> Terminate; footprint Button_Switch_THT:SW_DIP_SPSTx04_Slide_9.78x12.34mm_W7.62mm_P2.54mm -> Button_Switch_THT:SW_DIP_SPSTx03_Slide_9.78x9.8mm_W7.62mm_P2.54mm
- SW2: value INT -> SW_DIP_x08; footprint Button_Switch_THT:SW_DIP_SPSTx06_Slide_9.78x17.42mm_W7.62mm_P2.54mm -> Button_Switch_THT:SW_DIP_SPSTx08_Slide_9.78x22.5mm_W7.62mm_P2.54mm
- SW3: value Terminate -> I2C RST
- U1: value 74LS00 -> 74HCT688; footprint Package_DIP:DIP-14_W7.62mm_Socket_LongPads -> Package_DIP:DIP-20_W7.62mm_Socket
- U2: value 74LS85 -> 74LS245; footprint Package_DIP:DIP-16_W7.62mm_Socket_LongPads -> Package_DIP:DIP-20_W7.62mm_Socket
- U3: footprint Package_DIP:DIP-20_W7.62mm_Socket_LongPads -> Package_DIP:DIP-20_W7.62mm_Socket
- moved SW1 90.0 mm to (122.2, 57.9)
- moved R4 88.6 mm to (127.3, 38.9)
- moved R3 87.8 mm to (124.7, 38.9)
- moved R2 87.1 mm to (122.2, 38.9)
- moved C2 85.0 mm to (186.3, 42.7), turned to -90 degrees
- moved U2 73.5 mm to (190.8, 50.3), turned to 90 degrees
- moved SW3 71.7 mm to (161.5, 85.9)
- moved U1 54.3 mm to (190.8, 121.4)
- moved C1 52.2 mm to (186.9, 113.8)
- moved R5 48.5 mm to (176.8, 103.6)
- moved R6 42.3 mm to (127.3, 64.3)
- moved R7 37.3 mm to (124.7, 64.3)
- moved R8 32.9 mm to (122.2, 64.3)
- moved U3 28.7 mm to (156.5, 50.3)
- moved C3 27.8 mm to (152.0, 42.7)
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- renumbered C4 to C10, C5 to C11, J1 to J3
Connections:
- net /A_{0} renamed A_{0}
- net /A_{10} renamed A_{10}
- net /A_{11} renamed A_{11}
- net /A_{12} renamed A_{12}
- net /A_{13} renamed A_{13}
- net /A_{14} renamed A_{14}
- net /A_{15} renamed A_{15}
- net /A_{8} renamed A_{8}
- net /A_{9} renamed A_{9}
- J3 pad c8: /~{INTA} -> /INTA
- R1 pad 2: /B_{4} -> /~{INT}
- R2 pad 2: /B_{5} -> Net-(R2-Pad2)
- R3 pad 2: /B_{6} -> Net-(R3-Pad2)
- R4 pad 2: /B_{7} -> Net-(R4-Pad2)
- R5 pad 2: /~{INT} -> /INTA_~{EN}
- SW1 pad 1: GND -> /SDA
- SW1 pad 2: GND -> /SCL
- SW1 pad 3: GND -> /~{INT_{I2C}}
- SW1 pad 4: GND -> Net-(R4-Pad2)
- SW1 pad 5: /B_{7} -> Net-(R3-Pad2)
- SW1 pad 6: /B_{6} -> Net-(R2-Pad2)
- SW2 pad 1: /RST_{5.5} -> GND
- SW2 pad 10: /INT_{I2C} -> /B_{6}
- SW2 pad 11: /INT_{I2C} -> /B_{5}
- SW2 pad 12: /INT_{I2C} -> /B_{4}
- SW2 pad 2: /RST_{6.5} -> GND
- SW2 pad 3: /RST_{7.5} -> GND
- SW2 pad 4: /RST_{5.5} -> GND
- SW2 pad 5: /RST_{6.5} -> GND
- SW2 pad 6: /RST_{7.5} -> GND
- SW2 pad 7: /INT -> GND
- SW2 pad 8: /INT -> GND
- SW2 pad 9: /INT -> /B_{7}
- SW3 pad 1: /SDA -> /RST_{5.5}
- SW3 pad 2: /SCL -> /RST_{6.5}
- SW3 pad 3: /~{INT_{I2C}} -> /RST_{7.5}
- SW3 pad 4: Net-(R8-Pad2) -> /RST
- SW3 pad 5: Net-(R7-Pad2) -> /RST
- SW3 pad 6: Net-(R6-Pad2) -> /RST
- U1 pad 1: /a=b -> GND
- U1 pad 10: /~{INT} -> GND
- U1 pad 11: /IOWR -> /B_{4}
- U1 pad 12: /~{IOR} -> /A_{4}
- U1 pad 13: /~{IOW} -> /B_{5}
- U1 pad 14: GND -> /A_{5}
- U1 pad 2: /a=b -> GND
- U1 pad 3: /~{a=b} -> GND
- U1 pad 4: /~{INT_{I2C}} -> /B_{1}
- U1 pad 5: /~{INT_{I2C}} -> /A_{1}
- U1 pad 6: /INT_{I2C} -> /B_{2}
- U1 pad 7: VCC -> /A_{2}
- U1 pad 8: /INT -> /B_{3}
- U1 pad 9: /~{INT} -> /A_{3}
- U2 pad 1: /B_{7} -> /DIR_{2}
- U2 pad 10: /A_{4} -> GND
- U2 pad 11: /B_{5} -> Net-(U2-Pad11)
- U2 pad 12: /A_{5} -> Net-(U2-Pad12)
- U2 pad 13: /A_{6} -> Net-(U2-Pad13)
- U2 pad 14: /B_{6} -> Net-(U2-Pad14)
- U2 pad 15: /A_{7} -> Net-(U2-Pad15)
- U2 pad 16: VCC -> Net-(U2-Pad16)
- U2 pad 2: GND -> D_{0}
- U2 pad 3: /IOWR -> D_{1}
- U2 pad 4: GND -> D_{2}
- U2 pad 5: /a>b -> D_{3}
- U2 pad 6: /a=b -> D_{4}
- U2 pad 7: /a<b -> D_{5}
- U2 pad 8: GND -> D_{6}
- U2 pad 9: /B_{4} -> D_{7}
- U3 pad 11: D_{3} -> Net-(U2-Pad15)
- U3 pad 12: D_{4} -> Net-(U2-Pad14)
- U3 pad 13: D_{5} -> Net-(U2-Pad13)
- U3 pad 14: D_{6} -> Net-(U2-Pad12)
- U3 pad 15: D_{7} -> Net-(U2-Pad11)
- U3 pad 17: /~{a=b} -> /~{CS}
- U3 pad 4: unconnected-(U3-Pad4) -> /~{IACK}
- U3 pad 7: D_{0} -> Net-(U2-Pad18)
- U3 pad 8: D_{1} -> Net-(U2-Pad17)
- U3 pad 9: D_{2} -> Net-(U2-Pad16)
Routing:
- net VCC: track 330.0 -> 585.7 mm
- net /~{IACK}: track 0.00 -> 93.9 mm, vias 0 -> 1
- net A_{0}: track 55.0 -> 144.8 mm, vias 1 -> 2
- net /~{INT_{I2C}}: track 98.3 -> 18.2 mm
- net /IOWR: track 79.2 -> 0.00 mm, vias 1 -> 0
- net /~{CS}: track 0.00 -> 73.9 mm, vias 0 -> 1
- net /a=b: track 65.4 -> 0.00 mm, vias 1 -> 0
- net /A_{1}: track 0.00 -> 62.2 mm
- net /RST: track 0.00 -> 61.0 mm
- net /INTA: track 0.00 -> 57.5 mm, vias 0 -> 2
- net /INTR: track 0.00 -> 56.2 mm
- net /B_{3}: track 0.00 -> 53.2 mm
- net /~{INT}: track 24.6 -> 76.8 mm, vias 0 -> 1
- net /A_{2}: track 0.00 -> 50.7 mm
- net /A_{3}: track 0.00 -> 50.3 mm
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Other:
- board text added: "0V"
- board text added: "1"
- board text added: "BFZ/MFA B I2C-Busmaster"
- board text added: "EEPROM"
- board text added: "GND +5V SDA SCL"
- board text added: "GND +5V SDA SCL ~{INT_{I2C}}"
- board text added: "INTA ~{EN}"
- board text added: "INTR"
- board text added: "RST 5.5"
- board text added: "RST 6.5"
- board text added: "RST 7.5"
- board text added: "RTC"
- board text added: "SCL"
- board text removed: "GND"
