File: MFA_I2C/MFA_I2C.kicad_sch (KiCad schematic)
At the start: 22 parts, among them J1 DIN41612_02x32_AC, J2 Conn_02x04_Odd_Even, SW1 Terminate, SW2 ADR, SW3 INT, U1 74LS00, U2 74LS85, U3 PCF8584, X1 ACO-3MHz-A

Commit message: changed
Parts:
- removed R1, R2, R3, R4: 4k7, Resistor_THT:R_Axial_DIN0207_L6.3mm_D2.5mm_P10.16mm_Horizontal, symbol Device:R
- removed U1: 74LS00, Package_DIP:DIP-14_W7.62mm_Socket_LongPads, symbol 74xx:74LS00
- removed U2: 74LS85, Package_DIP:DIP-16_W7.62mm_Socket_LongPads, symbol 74xx:74LS85
- added C1, C2: 4.7uF, Capacitor_THT:C_Radial_D4.0mm_H5.0mm_P1.50mm, symbol Device:C_Polarized_Small
- added C6: 0.1uF, Capacitor_THT:C_Rect_L4.6mm_W2.0mm_P2.50mm_MKS02_FKP02, symbol Device:C_Small
- added H1, H2, H3, H4: MountingHole_Pad, MountingHole:MountingHole_3.2mm_M3_ISO14580_Pad, symbol Mechanical:MountingHole_Pad
- added J2: Conn_01x05, Connector_PinHeader_2.54mm:PinHeader_1x05_P2.54mm_Vertical, symbol Connector_Generic:Conn_01x05
- added RN1: 5k6, Resistor_THT:R_Array_SIP9, symbol Device:R_Network08
- added SW1: SW_DIP_x08, Button_Switch_THT:SW_DIP_SPSTx08_Slide_9.78x22.5mm_W7.62mm_P2.54mm, symbol Switch:SW_DIP_x08
- added U1: 74HCT688, symbol 74xx:74LS688
- added U2: 74LS245, Package_DIP:DIP-20_W7.62mm_Socket, symbol 74xx:74LS245
- added U3: GAL16V8A, Package_DIP:DIP-20_W7.62mm_Socket, symbol Logic_Programmable:GAL16V8
- J3: renamed from J2; value Conn_02x04_Odd_Even -> Conn_02x03_Odd_Even; footprint Connector_IDC:IDC-Header_2x04_P2.54mm_Horizontal -> Connector_IDC:IDC-Header_2x03_P2.54mm_Horizontal; symbol Connector_Generic:Conn_02x04_Odd_Even -> Connector_Generic:Conn_02x03_Odd_Even
- SW2: value ADR -> I2C RST
- SW3: value INT -> Master INT; footprint Button_Switch_THT:SW_DIP_SPSTx06_Slide_9.78x17.42mm_W7.62mm_P2.54mm -> Button_Switch_THT:SW_DIP_SPSTx04_Slide_9.78x12.34mm_W7.62mm_P2.54mm; symbol Switch:SW_DIP_x06 -> Switch:SW_DIP_x04
- U4: renamed from U3; footprint Package_DIP:DIP-20_W7.62mm_Socket_LongPads -> Package_DIP:DIP-20_W7.62mm_Socket
- renumbered C1 to C7, C2 to C8, R8 to R1, R5 to R2, R6 to R3, R7 to R4, SW1 to SW4
Connections:
- net A_{1}: now also U1.5 (R1)
- net A_{2}: now also U1.7 (R2)
- net A_{3}: now also U1.9 (R3)
- net A_{4}: now also U1.12 (R4)
- net A_{5}: now also U1.14 (R5)
- net A_{6}: now also U1.16 (R6)
- net A_{7}: now also U1.18 (R7)
- net B_{4}: now also RN1.6 (R5), SW1.12, U1.11 (P4); no longer SW2.8
- net B_{5}: now also RN1.7 (R6), SW1.11, U1.13 (P5); no longer SW2.7
- net B_{6}: now also RN1.8 (R7), SW1.10, U1.15 (P6); no longer SW2.6
- net B_{7}: now also RN1.9 (R8), SW1.9, U1.17 (P7); no longer SW2.5
- net D_{0}: now also U2.18 (B0); no longer U4.7 (D0)
- net D_{1}: now also U2.17 (B1); no longer U4.8 (D1)
- net D_{2}: now also U2.16 (B2); no longer U4.9 (D2)
- net D_{3}: now also U2.15 (B3); no longer U4.11 (D3)
- net D_{4}: now also U2.14 (B4); no longer U4.12 (D4)
- net D_{5}: now also U2.13 (B5); no longer U4.13 (D5)
- net D_{6}: now also U2.12 (B6); no longer U4.14 (D6)
- net D_{7}: now also U2.11 (B7); no longer U4.15 (D7)
- net GND: now also J3.4 (Pin_4), J3.6 (Pin_6), C1.2, C2.2, C6.2, H1.1, H2.1, H3.1, H4.1, J2.5 (Pin_5), SW1.1, SW1.2, SW1.3, SW1.4, SW1.5, SW1.6, SW1.7, SW1.8, U1.1 (G), U1.10 (GND), U1.2 (P0), U1.3 (R0), U2.10 (GND), U3.10 (GND); no longer J3.7 (Pin_7), J3.8 (Pin_8), SW2.1, SW2.2, SW2.3, SW2.4
- net INTR: now also SW3.4
- net RST_{5.5}: now also SW2.1; no longer SW3.4
- net RST_{6.5}: now also SW2.2; no longer SW3.5
- net RST_{7.5}: now also SW2.3; no longer SW3.6
- net SCL: now also J3.5 (Pin_5), J2.3 (Pin_3); no longer J3.4 (Pin_4)
- net SDA: now also J2.2 (Pin_2)
- net VCC: now also C1.1, C2.1, C6.1, J2.1 (Pin_1), RN1.1 (common), U1.20 (VCC), U3.20 (VCC); no longer J3.2 (Pin_2)
- net ~{INT_{I2C}}: now also J3.2 (Pin_2), J2.4 (Pin_4), U3.7 (I7); no longer J3.5 (Pin_5)
- net ~{INT}: now also U3.6 (I6)
- net ~{IOR}: now also U3.4 (I4); no longer U4.16 (~{RD})
- net ~{IOW}: now also U3.5 (I5); no longer U4.18 (~{WR})
- net INT: now reaches SW3.7, SW3.8
- net INT: now also SW3.5, SW3.6, U3.18 (IO2); no longer SW3.9
- net ~{IACK}: now reaches U4.4 (~{IACK})
- net ~{IACK}: now also U3.12 (IO8)
- net ~{INTA} renamed INTA
- net INTA: now also U3.3 (I3)
- net ~{a=b} renamed ~{CS}
- net ~{CS}: now also U3.15 (IO5)
- new net: U2.5 (A3), U4.11 (D3)
- new net: U2.6 (A4), U4.12 (D4)
- new net: U2.7 (A5), U4.13 (D5)
- new net: U2.8 (A6), U4.14 (D6)
- new net: U2.9 (A7), U4.15 (D7)
- new net: U2.2 (A0), U4.7 (D0)
- new net: U2.3 (A1), U4.8 (D1)
- new net: U2.4 (A2), U4.9 (D2)
- new net B_{0}: RN1.2 (R1), SW1.16
- new net B_{1}: RN1.3 (R2), SW1.15, U1.4 (P1)
- new net B_{2}: RN1.4 (R3), SW1.14, U1.6 (P2)
- new net B_{3}: RN1.5 (R4), SW1.13, U1.8 (P3)
- new net DIR_{2}: U2.1 (A->B), U3.16 (IO4)
- new net RST: SW2.5, SW2.6, SW2.7, SW2.8, U3.19 (IO1)
- new net ~{ADR}: U1.19 (P=R), U3.2 (I2)
- new net ~{CS_{2}}: U2.19 (CE), U3.17 (I03)
- new net ~{RD}: U3.14 (IO6), U4.16 (~{RD})
- new net ~{WR}: U3.13 (IO7), U4.18 (~{WR})
- no-connect marks 8 -> 11
Other:
- added sheet Untitled Sheet (untitled.kicad_sch)
- note added: "Addr Compare"
- note added: "BUS"
- note added: "Clock Register S24 S23 S22 S21 S20 f_{clk} f_{SCL} 0 x x 0 0 3MHz 90kHz Control PIN ESO ES1 ES2 ENI STA STO ACK Status PIN 0 STS BER AD0/LRB AAS LAB ~{BB}"
- note added: "ESO=0 A0 ES1 ES2 ~{IACK} Function 1 0 x 1 R/W S1: control 0 0 0 1 R/W S0: own address 0 0 1 1 R/W S3: interrupt vector 0 1 0 1 R/W S2: clock register ESO=1 A0 ES1 ES2 ~{IACK} Function 1 0 x 1 W S1: control 1 0 x 1 R S1: status 0 0 0 1 R/W S0: data 0 0 1 1 R/W S3: interrupt vector x 0 x 0 R S3: interrupt vector ACK cycle"
- note added: "I2C Connector"
- note added: "Interrupt Select"
- note added: "RST = !I2C; RST.oe = !INT; INTR = !INT; INTR.oe = !INT; !CS2 = (!ADR & (!IOR # !IOW)) # (INTA & !INT); DIR2 = (!ADR & !IOR) # (INTA & !INT); !CS = !ADR # (INTA & !INT); !RD = !CS2 & !IOR; !WR = !CS2 & !IOW; !IACK = !CS2 & (INTA & !INT);"
- note added: "external"
- note added: "internal"
- note removed: "Adress compare"
- note removed: "Interrupt"
- company: (none) -> Non commercial use only !
- title: (none) -> MFA I2C Busmaster
- moved on the sheet: C4, C5, C7, C8, R1, R4, SW4, U4, X1

Commit message: next version
Parts:
- removed J2: Conn_01x05, Connector_PinHeader_2.54mm:PinHeader_1x05_P2.54mm_Vertical, symbol Connector_Generic:Conn_01x05
- removed J3: Conn_02x03_Odd_Even, Connector_IDC:IDC-Header_2x03_P2.54mm_Horizontal, symbol Connector_Generic:Conn_02x03_Odd_Even
- removed U3: GAL16V8A, Package_DIP:DIP-20_W7.62mm_Socket, symbol Logic_Programmable:GAL16V8
- added C5, C6: 0.1uF, Capacitor_THT:C_Rect_L4.6mm_W2.0mm_P2.50mm_MKS02_FKP02, symbol Device:C_Small
- added R5: 10k, Resistor_THT:R_Axial_DIN0207_L6.3mm_D2.5mm_P7.62mm_Horizontal, symbol Device:R
- added U4: 74LS04, Package_DIP:DIP-14_W7.62mm_Socket, symbol 74xx:74LS04
- added U5, U6: 74LS00, Package_DIP:DIP-14_W7.62mm_Socket, symbol 74xx:74LS00
- R1, R2, R3, R4: footprint Resistor_THT:R_Axial_DIN0207_L6.3mm_D2.5mm_P10.16mm_Horizontal -> Resistor_THT:R_Axial_DIN0207_L6.3mm_D2.5mm_P7.62mm_Horizontal
- SW3: renamed from SW2; footprint Button_Switch_THT:SW_DIP_SPSTx04_Slide_9.78x12.34mm_W7.62mm_P2.54mm -> Button_Switch_THT:SW_DIP_SPSTx03_Slide_9.78x9.8mm_W7.62mm_P2.54mm; symbol Switch:SW_DIP_x04 -> Switch:SW_DIP_x03
- SW4: renamed from SW3; footprint Button_Switch_THT:SW_DIP_SPSTx04_Slide_9.78x12.34mm_W7.62mm_P2.54mm -> Button_Switch_THT:SW_DIP_SPSTx05_Slide_9.78x14.88mm_W7.62mm_P2.54mm; symbol Switch:SW_DIP_x04 -> Switch:SW_DIP_x05
- U1: footprint (none) -> Package_DIP:DIP-20_W7.62mm_Socket
- renumbered C3 to C1, C7 to C10, C8 to C11, C1 to C12, C2 to C13, C4 to C2, C5 to C3, C6 to C4, J1 to J3, SW4 to SW1, SW1 to SW2, U4 to U3
Connections:
- net ~{RD} is gone; now on net ~{IOR}: U3.16 (~{RD})
- net ~{WR} is gone; now on net ~{IOW}: U3.18 (~{WR})
- net B_{0}: now also RN1.9 (R8); no longer RN1.2 (R1)
- net B_{1}: now also RN1.8 (R7); no longer RN1.3 (R2)
- net B_{2}: now also RN1.7 (R6); no longer RN1.4 (R3)
- net B_{3}: now also RN1.6 (R5); no longer RN1.5 (R4)
- net B_{4}: now also RN1.5 (R4); no longer RN1.6 (R5)
- net B_{5}: now also RN1.4 (R3); no longer RN1.7 (R6)
- net B_{6}: now also RN1.3 (R2); no longer RN1.8 (R7)
- net B_{7}: now also RN1.2 (R1); no longer RN1.9 (R8)
- net DIR_{2}: now also U5.11
- net D_{0}: now also U2.2 (A0); no longer U2.18 (B0)
- net D_{1}: now also U2.3 (A1); no longer U2.17 (B1)
- net D_{2}: now also U2.4 (A2); no longer U2.16 (B2)
- net D_{3}: now also U2.5 (A3); no longer U2.15 (B3)
- net D_{4}: now also U2.6 (A4); no longer U2.14 (B4)
- net D_{5}: now also U2.7 (A5); no longer U2.13 (B5)
- net D_{6}: now also U2.8 (A6); no longer U2.12 (B6)
- net D_{7}: now also U2.9 (A7); no longer U2.11 (B7)
- net GND: now also SW4.5, C5.2, C6.2, U4.14 (VCC), U5.7 (GND), U6.7 (GND)
- net INT: now also SW4.10, SW4.9, U4.12; no longer SW4.5, SW4.6
- net INTA: now also U6.2
- net RST: now also SW3.4, U4.2; no longer SW3.7, SW3.8
- net VCC: now also U2.20 (VCC), C5.1, C6.1, R5.1, U4.7 (GND), U5.14 (VCC), U6.14 (VCC)
- net ~{ADR}: now also U6.10
- net ~{CS}: now also U6.11
- net ~{IACK}: now also U5.2, U6.3, U6.9
- net ~{INT_{I2C}}: now also U4.1
- net ~{INT}: now also U4.13
- net ~{IOR}: now also U5.1
- net ~{IOW}: now also U5.4
- net at U3.11 (D3): now also U2.15 (B3); no longer U2.5 (A3)
- net at U3.12 (D4): now also U2.14 (B4); no longer U2.6 (A4)
- net at U3.13 (D5): now also U2.13 (B5); no longer U2.7 (A5)
- net at U3.14 (D6): now also U2.12 (B6); no longer U2.8 (A6)
- net at U3.15 (D7): now also U2.11 (B7); no longer U2.9 (A7)
- net at U3.7 (D0): now also U2.18 (B0); no longer U2.2 (A0)
- net at U3.8 (D1): now also U2.17 (B1); no longer U2.3 (A1)
- net at U3.9 (D2): now also U2.16 (B2); no longer U2.4 (A2)
- net ~{CS_{2}} renamed ~{CE_{2}}
- net ~{CE_{2}}: now also U5.8
- new net ADR#IACK: U5.10, U5.13, U6.12, U6.13, U6.8
- new net INTA_~{EN}: R5.2, SW4.6, U6.1
- new net IOR#IACK: U5.12, U5.3, U6.4, U6.5
- new net IOR#IOW#IACK: U5.6, U5.9
- new net ~{IOR#IACK}: U5.5, U6.6
- no-connect marks 11 -> 6
Other:
- removed sheet Untitled Sheet
- added sheet  Application (I2C_Application.kicad_sch)
- note added: "DIR_{2}=~{(ADR#IACK)&(IOR#IACK)}"
- note added: "Decoder"
- note added: "L: BUS<-PCF H: BUS->PCF"
- note added: "~{CE_{2}}=(ADR#IACK)&(IOR#IACK#IOW)"
- note added: "~{CS}=ADR#IACK"
- note removed: "BUS"
- note removed: "Clock Register S24 S23 S22 S21 S20 f_{clk} f_{SCL} 0 x x 0 0 3MHz 90kHz Control PIN ESO ES1 ES2 ENI STA STO ACK Status PIN 0 STS BER AD0/LRB AAS LAB ~{BB}"
- note removed: "ESO=0 A0 ES1 ES2 ~{IACK} Function 1 0 x 1 R/W S1: control 0 0 0 1 R/W S0: own address 0 0 1 1 R/W S3: interrupt vector 0 1 0 1 R/W S2: clock register ESO=1 A0 ES1 ES2 ~{IACK} Function 1 0 x 1 W S1: control 1 0 x 1 R S1: status 0 0 0 1 R/W S0: data 0 0 1 1 R/W S3: interrupt vector x 0 x 0 R S3: interrupt vector ACK cycle"
- note removed: "I2C Connector"
- note removed: "RST = !I2C; RST.oe = !INT; INTR = !INT; INTR.oe = !INT; !CS2 = (!ADR & (!IOR # !IOW)) # (INTA & !INT); DIR2 = (!ADR & !IOR) # (INTA & !INT); !CS = !ADR # (INTA & !INT); !RD = !CS2 & !IOR; !WR = !CS2 & !IOW; !IACK = !CS2 & (INTA & !INT);"
- moved on the sheet: C1, C10, C11, C12, C13, C2, C3, C4, H1, H2, H3, H4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
